File: Lidar/Lidar_teensy/board1.brd (EAGLE design)
At the start: 101.5 x 76 mm, 43 parts, among them IC1 DS3231/SO, Q4 IPS6021R, U1 INA219BIDCNT

Commit message: updated route, rtc alarm update
Parts:
- added LED1: 120, adafruit:CHIPLED_1206
- added R15: 50k, microbuilder:0805-NO
- added R16: 120R, microbuilder:0805-NO
- added S2: TL32PO, switch:TL3XPO
- added SV1, SV2: (no value), con-lstb:MA05-1
- added SV3: (no value), con-lstb:MA09-1
- C3: device SparkFun-Passives:VISHAY_C -> SparkFun-Passives:EIA7343
- moved Q4 24.2 mm to (59.8, 14.1), turned to 180 degrees
- moved C2 24.0 mm to (45.8, 26.0), turned to 90 degrees
- moved LIDAR 20.9 mm to (47.5, 7.87), turned to 180 degrees
- moved R6 17.0 mm to (44.6, 18.7), turned to 0 degrees
- moved R4 16.7 mm to (44.6, 22.0), turned to 0 degrees
- moved D5 16.5 mm to (59.1, 24.6), turned to 0 degrees
- moved R21 15.9 mm to (58.6, 22.5), turned to 180 degrees
- moved U1 13.8 mm to (36.4, 18.4)
- moved X2 13.6 mm to (33.5, 8.29)
- moved U$2 11.9 mm to (52.8, 20.1)
- moved R11 11.6 mm to (43.0, 48.4), turned to 0 degrees
- moved R10 8.72 mm to (43.8, 50.4)
- moved R3 7.54 mm to (35.8, 24.8), turned to 180 degrees
- moved U$3 1.02 mm to (17.7, 19.4)
- moved H6 0.32 mm to (96.4, 70.3)
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Connections:
- removed net !RTC_RST: IC1.4
- removed net +VIN: Q4.5, R3.1, U1.1
- removed net -VIN: R3.2, U$2.P$1, U1.2
- new net +9V: S2.3, X2.1
- new net +VCC: R3.1, S2.2, U1.1
- new net N$12: SV3.4, U$1.SAG
- new net N$13: SV3.3, U$1.CSM
- new net N$14: SV3.2, U$1.SDAOG
- new net N$15: Q4.5, U$2.P$1
- new net N$16: SV3.1, U$1.SDOM
- new net N$17: SV2.1, U$1.DEN
- new net N$18: SV2.2, U$1.INT2
- new net N$19: SV2.3, U$1.INT1
- new net N$20: SV2.4, U$1.DRDY
- new net N$21: SV2.5, U$1.INTM
- new net N$22: SV1.5, XBEE.RST
- new net N$3: JP1.6, R16.1
- new net N$6: LED1.A, R16.2
- new net N$8: SV3.8, U$1.3V3
- net +3V3: now also R15.2
- net 5V: now also SV1.1, SV3.9; no longer JP1.VIN
- net 5V_OUT: now also JP1.VIN
- net GND: now also C3.C, IC1.10, IC1.11, IC1.12, IC1.5, IC1.6, IC1.7, IC1.8, IC1.9, LED1.C, SV1.2, SV3.7; no longer C3.-
- net RX_X: now also SV1.3
- net SCL_P: now also SV3.6
- net SDA_P: now also SV3.5
- net SQW: now also R15.1
- net TX_X: now also SV1.4
- net VBAT: now also C3.A; no longer C3.+
- net VCC: now also R3.2, U1.2; no longer X2.1
Routing:
- net 5V_OUT: track 18.4 -> 81.1 mm
- net +VCC: track 0.00 -> 54.7 mm, vias 0 -> 1
- net +VIN: track 37.2 -> 0.00 mm, vias 2 -> 0
- net N$11: track 46.4 -> 12.5 mm, vias 2 -> 0
- net 5V: track 176.4 -> 143.3 mm, vias 2 -> 0
- net VCC: track 19.3 -> 42.9 mm
- net -VIN: track 15.2 -> 0.00 mm
- net SCL_P: track 69.7 -> 83.4 mm, vias 2 -> 1
- net SDA_P: track 91.2 -> 77.5 mm, vias 2 -> 1
- net N$2: track 19.3 -> 5.99 mm, vias 2 -> 0
- net +9V: track 0.00 -> 10.0 mm
- net N$1: track 16.8 -> 7.07 mm, vias 2 -> 0
- net N$3: track 0.00 -> 8.52 mm
- net N$15: track 0.00 -> 8.51 mm
- net N$4: track 13.8 -> 6.27 mm
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- added copper zone on layer 1, net N$23
- removed copper zone on layer 1, net N$12
- removed copper zone on layer 16, net N$13
- removed copper zone on layer 16, net N$14
- removed copper zone on layer 1, net N$3
- removed copper zone on layer 1, net N$6
- removed copper zone on layer 1, net N$8
Other:
- board text added: "07-04-2018 mad"
- board text removed: "+"
- board text removed: "06-27-2018 mad"
