File: Lidar/Lidar_teensy/board1.sch (EAGLE design)
At the start: 43 parts, among them IC1 DS3231/SO, Q4 IPS6021R, U1 INA219BIDCNT

Commit message: updated route, rtc alarm update
Parts:
- added LED1: 120, adafruit:LEDCHIPLED_1206
- added R15: 50k, microbuilder:RESISTOR0805_NOOUTLINE
- added R16: 120R, microbuilder:RESISTOR0805_NOOUTLINE
- added S2: TL32PO, switch:TL32PO
- added SV1, SV2: (no value), con-lstb:MA05-1
- added SV3: (no value), con-lstb:MA09-1
- C3: device SparkFun-Passives:CAP_POLSMD -> SparkFun-Passives:CAP_POL7343
Connections:
- removed net !RTC_RST: IC1./RST
- removed net +VIN: Q4.OUT, R3.1, U1.VIN+
- removed net -VIN: R3.2, U$2.1, U1.VIN-
- new net +9V: S2.S, X2-1.KL
- new net +VCC: R3.1, S2.P, U1.VIN+
- new net N$12: SV3.4, U$1.SAG
- new net N$13: SV3.3, U$1.CSM
- new net N$14: SV3.2, U$1.SDOAG
- new net N$15: Q4.OUT, U$2.1
- new net N$16: SV3.1, U$1.SDOM
- new net N$17: SV2.1, U$1.DEN
- new net N$18: SV2.2, U$1.INT2
- new net N$19: SV2.3, U$1.INT1
- new net N$20: SV2.4, U$1.DRDY
- new net N$21: SV2.5, U$1.INTM
- new net N$22: SV1.5, XBEE.RST
- new net N$3: JP1.6*, R16.1
- new net N$6: LED1.A, R16.2
- new net N$8: SV3.8, U$1.3V3
- net +3V3: now also R15.2
- net 5V: now also SV1.1, SV3.9; no longer JP1.VIN
- net 5V_OUT: now also JP1.VIN
- net GND: now also IC1.NC, IC1.NC1, IC1.NC2, IC1.NC3, IC1.NC4, IC1.NC5, IC1.NC6, IC1.NC7, LED1.C, SV1.2, SV3.7
- net RX_X: now also SV1.3
- net SCL_P: now also SV3.6
- net SDA_P: now also SV3.5
- net SQW: now also R15.1
- net TX_X: now also SV1.4
- net VCC: now also R3.2, U1.VIN-; no longer X2-1.KL
Other:
- moved on the sheet: R10, R11, R12, R13, R14, R7, R8, R9, U$11, U$12, U$7, U$8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
