File: loraDue/Arabica/m0_lora.brd (EAGLE design)
At the start: 51.6 x 41.3 mm, 38 parts, among them J1 S2B-PH-SM4-TB(LF)(SN)

Commit message: finalized board details
Parts:
- renumbered C1 to 1UF, C2 to 0.1UF, Q1 to PNP, R1 to 47K, R2 to 4.7K, R3 to 4.7K2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
Other:
- outline, holes or cut-outs redrawn
- board text added: "VIN"
